Commit message: improved GUI and error handling, added Websockets

File: install/my_robot_description/share/my_robot_description/urdf/my_robot.urdf.xacro (robot description, xacro)
@@ -1,7 +1,13 @@
 <?xml version="1.0"?>
 <robot name="my_robot_arm" xmlns:xacro="http://www.ros.org/wiki/xacro">
+  <xacro:arg name="controller_config_path" default=""/>
   <xacro:property name="package_path" value="$(find my_robot_description)" />
-  <!-- Links and Joints are here... they are correct and have been omitted for brevity -->
   <link name="world" />
+  <link name="base_footprint" />
+  <joint name="base_footprint_joint" type="fixed">
+    <parent link="world"/>
+    <child link="base_footprint"/>
+    <origin xyz="0 0 0.01" rpy="0 0 0"/>
+  </joint>
   <link name="base">
     <visual>
@@ -18,8 +24,13 @@
     </collision>
     <inertial>
-      <mass value="0.9"/>
+      <mass value="2.5"/>
       <inertia ixx="0.01" ixy="0" ixz="0" iyy="0.01" iyz="0" izz="0.01"/>
     </inertial>
   </link>
+  <joint name="base_joint" type="fixed">
+    <parent link="base_footprint"/>
+    <child link="base"/>
+    <origin xyz="0 0 0" rpy="0 0 0"/>
+  </joint>
   <link name="base_link">
     <visual>
@@ -36,5 +47,5 @@
     </collision>
     <inertial>
-      <mass value="0.5"/>
+      <mass value="1.5"/>
       <inertia ixx="0.01" ixy="0" ixz="0" iyy="0.01" iyz="0" izz="0.01"/>
     </inertial>
@@ -54,5 +65,5 @@
     </collision>
     <inertial>
-      <mass value="0.6"/>
+      <mass value="1.2"/>
       <inertia ixx="0.01" ixy="0" ixz="0" iyy="0.01" iyz="0" izz="0.01"/>
     </inertial>
@@ -72,5 +83,5 @@
     </collision>
     <inertial>
-      <mass value="0.4"/>
+      <mass value="1.0"/>
       <inertia ixx="0.01" ixy="0" ixz="0" iyy="0.01" iyz="0" izz="0.01"/>
     </inertial>
@@ -90,6 +101,6 @@
     </collision>
     <inertial>
-      <mass value="0.3"/>
-      <inertia ixx="0.01" ixy="0" ixz="0" iyy="0.01" iyz="0" izz="0.01"/>
+      <mass value="0.8"/>
+      <inertia ixx="0.001" ixy="0" ixz="0" iyy="0.001" iyz="0" izz="0.001"/>
     </inertial>
   </link>
@@ -109,28 +120,7 @@
     <inertial>
       <mass value="0.5"/>
-      <inertia ixx="0.01" ixy="0" ixz="0" iyy="0.01" iyz="0" izz="0.01"/>
+      <inertia ixx="0.001" ixy="0" ixz="0" iyy="0.001" iyz="0" izz="0.001"/>
     </inertial>
   </link>
-  <link name="link_5_wrist_roll">
-    <inertial>
-      <mass value="0.1"/>
-      <inertia ixx="0.001" ixy="0.0" ixz="0.0" iyy="0.001" iyz="0.0" izz="0.001"/>
-    </inertial>
-    <visual>
-      <geometry>
-        <cylinder length="0.02" radius="0.02"/>
-      </geometry>
-    </visual>
-    <collision>
-      <geometry>
-        <cylinder length="0.02" radius="0.02"/>
-      </geometry>
-    </collision>
-  </link>
-  <joint name="world_to_base_fixed" type="fixed">
-    <parent link="world"/>
-    <child link="base"/>
-    <origin rpy="0 0 0" xyz="0 0 0"/>
-  </joint>
   <joint name="joint1" type="revolute">
     <parent link="base"/>
@@ -165,11 +155,4 @@
     <child link="link_4_wrist"/>
     <origin rpy="3.141592653589793 0 0" xyz="-0.018 0 -0.12"/>
-    <axis xyz="1 0 0"/>
-    <limit effort="100" lower="-3.14" upper="3.14" velocity="1.0"/>
-  </joint>
-  <joint name="joint6" type="revolute">
-    <parent link="link_4_wrist"/>
-    <child link="link_5_wrist_roll"/>
-    <origin rpy="0 0 0" xyz="0 0 0.05"/>
     <axis xyz="0 1 0"/>
     <limit effort="100" lower="-3.14" upper="3.14" velocity="1.0"/>
@@ -204,17 +187,8 @@
       <state_interface name="velocity"/>
     </joint>
-    <joint name="joint6">
-      <command_interface name="position"/>
-      <state_interface name="position"/>
-      <state_interface name="velocity"/>
-    </joint>
   </ros2_control>
-  <!-- =================================================================== -->
-  <!-- === THE FINAL FIX: ADD THE GAZEBO PLUGIN AND CONTROLLER CONFIG  === -->
-  <!-- This tag tells Gazebo to load the ros2_control plugin and where to find its parameters. -->
-  <!-- =================================================================== -->
-  <gazebo>
+   <gazebo>
     <plugin filename="libgazebo_ros2_control.so" name="gazebo_ros2_control">
-      <parameters>$(find my_robot_description)/config/my_robot_arm_controllers.yaml</parameters>
+      <parameters>$(arg controller_config_path)</parameters>
     </plugin>
   </gazebo>
