Commit message: fix: Adjust robot and gripper joint origins/rotations and update mesh paths to be relative.

File: install/visiona_bridge/share/visiona_bridge/urdf/visiona.urdf.xacro (robot description, xacro)
@@ -148,5 +148,5 @@
     </joint>
     <joint name="base_link_joint" type="revolute">
-        <origin xyz="0.0 0.0 0.0" rpy="0.0 0.0 0.0" />
+        <origin xyz="0.0 0.0 -0.001" rpy="0.0 0.0 0.0" />
         <parent link="base" />
         <child link="base_link" />
@@ -156,5 +156,5 @@
     </joint>
     <joint name="link_1_shoulder_joint" type="revolute">
-        <origin xyz="-0.0055 0 0.134 " rpy="0.0 0.0 0.0" />
+        <origin xyz="-0.0055 0 0.14 " rpy="0.0 0.0 0.0" />
         <parent link="base_link" />
         <child link="link_1_shoulder" />
@@ -172,5 +172,5 @@
     </joint>
     <joint name="link_3_wrist_joint" type="revolute">
-        <origin xyz="0 0 0.116 " rpy="0 0 3.14" />
+        <origin xyz="0 -0.119 0 " rpy="-1.57 0 0" />
         <parent link="link_2_elbow" />
         <child link="link_3_wrist" />

File: src/visiona_bridge/urdf/gripper.xacro (robot description, xacro)
@@ -6,5 +6,5 @@
                 <origin xyz="0 0 0" rpy="0 0 0" />
                 <geometry>
-                    <mesh filename="file:///home/farouk/ros2_ws/src/visiona_bridge/meshes/gripper_joint.stl"
+                    <mesh filename="../meshes/gripper_joint.stl"
                         scale="0.001 0.001 0.001" />
                 </geometry>
@@ -14,5 +14,5 @@
                 <origin xyz="0 0 0" rpy="0 0 0" />
                 <geometry>
-                    <mesh filename="file:///home/farouk/ros2_ws/src/visiona_bridge/meshes/gripper_joint.stl"
+                    <mesh filename="../meshes/gripper_joint.stl"
                         scale="0.001 0.001 0.001" />
                 </geometry>
@@ -27,4 +27,5 @@
             <child link="gripper_base" />
             <xacro:insert_block name="origin_block" />
+            <origin xyz="0 -0.085 0" rpy="3.14 0 0" />
             <axis xyz="0 1 0.0" />
             <limit lower="-3.0" upper="3.0" effort="100.0" velocity="10.0" />
@@ -35,5 +36,5 @@
                 <origin xyz="0 0 0" rpy="0 0 0" />
                 <geometry>
-                    <mesh filename="file:///home/farouk/ros2_ws/src/visiona_bridge/meshes/gripper_left_finger.stl"
+                    <mesh filename="../meshes/gripper_left_finger.stl"
                         scale="0.001 0.001 0.001" />
                 </geometry>
@@ -42,5 +43,5 @@
                 <origin xyz="0 0 0" rpy="0 0 0" />
                 <geometry>
-                    <mesh filename="file:///home/farouk/ros2_ws/src/visiona_bridge/meshes/gripper_left_finger.stl"
+                    <mesh filename="../meshes/gripper_left_finger.stl"
                         scale="0.001 0.001 0.001" />
                 </geometry>
@@ -55,5 +56,5 @@
                 <origin xyz="0 0 0" rpy="0 0 0" />
                 <geometry>
-                    <mesh filename="file:///home/farouk/ros2_ws/src/visiona_bridge/meshes/gripper_right_finger.stl"
+                    <mesh filename="../meshes/gripper_right_finger.stl"
                         scale="0.001 0.001 0.001" />
                 </geometry>
@@ -62,5 +63,5 @@
                 <origin xyz="0 0 0" rpy="0 0 0" />
                 <geometry>
-                    <mesh filename="file:///home/farouk/ros2_ws/src/visiona_bridge/meshes/gripper_right_finger.stl"
+                    <mesh filename="../meshes/gripper_right_finger.stl"
                         scale="0.001 0.001 0.001" />
                 </geometry>

File: src/visiona_bridge/urdf/visiona.urdf.xacro (robot description, xacro)
@@ -15,5 +15,5 @@
             <origin xyz="0 0 0 " rpy="0 0 0 " />
             <geometry>
-                <mesh filename="file:///home/farouk/ros2_ws/src/visiona_bridge/meshes/base.stl" scale="0.001 0.001 0.001" />
+                <mesh filename="../meshes/base.stl" scale="0.001 0.001 0.001" />
             </geometry>
         </visual>
@@ -58,5 +58,5 @@
             <origin xyz="0 0 0.075 " rpy="0 0 0 " />
             <geometry>
-                <mesh filename="file:///home/farouk/ros2_ws/src/visiona_bridge/meshes/base_link.stl"
+                <mesh filename="../meshes/base_link.stl"
                     scale="0.001 0.001 0.001" />
             </geometry>
@@ -78,5 +78,5 @@
             <origin xyz="0 0 0 " rpy="0 0 0 " />
             <geometry>
-                <mesh filename="file:///home/farouk/ros2_ws/src/visiona_bridge/meshes/link_1_shoulder.stl"
+                <mesh filename="../meshes/link_1_shoulder.stl"
                     scale="0.001 0.001 0.001" />
             </geometry>
@@ -98,5 +98,5 @@
             <origin xyz="0 0 0 " rpy="1.57 0 0 " />
             <geometry>
-                <mesh filename="file:///home/farouk/ros2_ws/src/visiona_bridge/meshes/link_2_elbow.stl"
+                <mesh filename="../meshes/link_2_elbow.stl"
                     scale="0.001 0.001 0.001" />
             </geometry>
@@ -118,5 +118,5 @@
             <origin xyz="0 0 0 " rpy="1.57 0 0 " />
             <geometry>
-                <mesh filename="file:///home/farouk/ros2_ws/src/visiona_bridge/meshes/link_3_wrist.stl"
+                <mesh filename="../meshes/link_3_wrist.stl"
                     scale="0.001 0.001 0.001" />
             </geometry>
@@ -148,5 +148,5 @@
     </joint>
     <joint name="base_link_joint" type="revolute">
-        <origin xyz="0.0 0.0 0.0" rpy="0.0 0.0 0.0" />
+        <origin xyz="0.0 0.0 -0.001" rpy="0.0 0.0 0.0" />
         <parent link="base" />
         <child link="base_link" />
@@ -156,5 +156,5 @@
     </joint>
     <joint name="link_1_shoulder_joint" type="revolute">
-        <origin xyz="-0.0055 0 0.134 " rpy="0.0 0.0 0.0" />
+        <origin xyz="-0.0055 0 0.14 " rpy="0.0 0.0 0.0" />
         <parent link="base_link" />
         <child link="link_1_shoulder" />
@@ -172,5 +172,5 @@
     </joint>
     <joint name="link_3_wrist_joint" type="revolute">
-        <origin xyz="0 0 0.116 " rpy="0 0 3.14" />
+        <origin xyz="0 -0.119 0 " rpy="-1.57 0 0" />
         <parent link="link_2_elbow" />
         <child link="link_3_wrist" />

Commit message: feat: Adjust URDF mesh paths, enable joint dynamics and gripper self-collision with friction, and remove unused installed model files.

File: install/visiona_bridge/share/visiona_bridge/urdf/visiona.urdf.xacro (robot description, xacro)
@@ -180,5 +180,5 @@
     </joint>
     <xacro:gripper parent_link="link_3_wrist">
-        <origin xyz="0 0 0.082" rpy="1.5707963 0 0" />
+        <origin xyz="0 -0.085 0" rpy="3.14 0 0" />
     </xacro:gripper>
     <xacro:include filename="visiona_gazebo.xacro" />

File: src/visiona_bridge/urdf/gripper.xacro (robot description, xacro)
@@ -6,5 +6,5 @@
                 <origin xyz="0 0 0" rpy="0 0 0" />
                 <geometry>
-                    <mesh filename="../meshes/gripper_joint.stl"
+                    <mesh filename="file:///home/farouk/ros2_ws/src/visiona_bridge/meshes/gripper_joint.stl"
                         scale="0.001 0.001 0.001" />
                 </geometry>
@@ -14,5 +14,5 @@
                 <origin xyz="0 0 0" rpy="0 0 0" />
                 <geometry>
-                    <mesh filename="../meshes/gripper_joint.stl"
+                    <mesh filename="file:///home/farouk/ros2_ws/src/visiona_bridge/meshes/gripper_joint.stl"
                         scale="0.001 0.001 0.001" />
                 </geometry>
@@ -27,8 +27,7 @@
             <child link="gripper_base" />
             <xacro:insert_block name="origin_block" />
-            <origin xyz="0 -0.085 0" rpy="3.14 0 0" />
             <axis xyz="0 1 0.0" />
             <limit lower="-3.0" upper="3.0" effort="100.0" velocity="10.0" />
-            <!-- <dynamics damping="10" friction="10" /> -->
+            <dynamics damping="10" friction="10" />
         </joint>
         <link name="left_finger_link">
@@ -36,5 +35,5 @@
                 <origin xyz="0 0 0" rpy="0 0 0" />
                 <geometry>
-                    <mesh filename="../meshes/gripper_left_finger.stl"
+                    <mesh filename="file:///home/farouk/ros2_ws/src/visiona_bridge/meshes/gripper_left_finger.stl"
                         scale="0.001 0.001 0.001" />
                 </geometry>
@@ -43,5 +42,5 @@
                 <origin xyz="0 0 0" rpy="0 0 0" />
                 <geometry>
-                    <mesh filename="../meshes/gripper_left_finger.stl"
+                    <mesh filename="file:///home/farouk/ros2_ws/src/visiona_bridge/meshes/gripper_left_finger.stl"
                         scale="0.001 0.001 0.001" />
                 </geometry>
@@ -56,5 +55,5 @@
                 <origin xyz="0 0 0" rpy="0 0 0" />
                 <geometry>
-                    <mesh filename="../meshes/gripper_right_finger.stl"
+                    <mesh filename="file:///home/farouk/ros2_ws/src/visiona_bridge/meshes/gripper_right_finger.stl"
                         scale="0.001 0.001 0.001" />
                 </geometry>
@@ -63,5 +62,5 @@
                 <origin xyz="0 0 0" rpy="0 0 0" />
                 <geometry>
-                    <mesh filename="../meshes/gripper_right_finger.stl"
+                    <mesh filename="file:///home/farouk/ros2_ws/src/visiona_bridge/meshes/gripper_right_finger.stl"
                         scale="0.001 0.001 0.001" />
                 </geometry>
@@ -78,5 +77,5 @@
             <axis xyz="0 0 1" />
             <limit lower="-1.0" upper="1" effort="100.0" velocity="10.0" />
-            <!-- <dynamics damping="10" friction="10" /> -->
+            <dynamics damping="10" friction="10" />
         </joint>
         <joint name="right_finger_joint" type="revolute">
@@ -86,5 +85,5 @@
             <axis xyz="0 0 1" />
             <limit lower="-1.0" upper="1" effort="100.0" velocity="10.0" />
-            <!-- <dynamics damping="10" friction="10" /> -->
+            <dynamics damping="10" friction="10" />
             <mimic joint="left_finger_joint" multiplier="-1" offset="0.0" />
         </joint>

File: src/visiona_bridge/urdf/visiona.urdf.xacro (robot description, xacro)
@@ -15,5 +15,5 @@
             <origin xyz="0 0 0 " rpy="0 0 0 " />
             <geometry>
-                <mesh filename="../meshes/base.stl" scale="0.001 0.001 0.001" />
+                <mesh filename="file:///home/farouk/ros2_ws/src/visiona_bridge/meshes/base.stl" scale="0.001 0.001 0.001" />
             </geometry>
         </visual>
@@ -58,5 +58,5 @@
             <origin xyz="0 0 0.075 " rpy="0 0 0 " />
             <geometry>
-                <mesh filename="../meshes/base_link.stl"
+                <mesh filename="file:///home/farouk/ros2_ws/src/visiona_bridge/meshes/base_link.stl"
                     scale="0.001 0.001 0.001" />
             </geometry>
@@ -78,5 +78,5 @@
             <origin xyz="0 0 0 " rpy="0 0 0 " />
             <geometry>
-                <mesh filename="../meshes/link_1_shoulder.stl"
+                <mesh filename="file:///home/farouk/ros2_ws/src/visiona_bridge/meshes/link_1_shoulder.stl"
                     scale="0.001 0.001 0.001" />
             </geometry>
@@ -98,5 +98,5 @@
             <origin xyz="0 0 0 " rpy="1.57 0 0 " />
             <geometry>
-                <mesh filename="../meshes/link_2_elbow.stl"
+                <mesh filename="file:///home/farouk/ros2_ws/src/visiona_bridge/meshes/link_2_elbow.stl"
                     scale="0.001 0.001 0.001" />
             </geometry>
@@ -118,5 +118,5 @@
             <origin xyz="0 0 0 " rpy="1.57 0 0 " />
             <geometry>
-                <mesh filename="../meshes/link_3_wrist.stl"
+                <mesh filename="file:///home/farouk/ros2_ws/src/visiona_bridge/meshes/link_3_wrist.stl"
                     scale="0.001 0.001 0.001" />
             </geometry>
@@ -153,5 +153,5 @@
         <axis xyz="0.0 0 1" />
         <limit lower="-3.14" upper="3.14" effort="100.0" velocity="10.0" />
-        <!-- <dynamics damping="10" friction="10" /> -->
+        <dynamics damping="10" friction="10" />
     </joint>
     <joint name="link_1_shoulder_joint" type="revolute">
@@ -161,5 +161,5 @@
         <axis xyz="1 0 0.0" />
         <limit lower="-1.57" upper="1.57" effort="100.0" velocity="10.0" />
-        <!-- <dynamics damping="10" friction="10" /> -->
+        <dynamics damping="10" friction="10" />
     </joint>
     <joint name="link_2_elbow_joint" type="revolute">
@@ -169,5 +169,5 @@
         <axis xyz="1 0 0.0" />
         <limit lower="-3.14" upper="3.14" effort="100.0" velocity="10.0" />
-        <!-- <dynamics damping="10" friction="10" /> -->
+        <dynamics damping="10" friction="10" />
     </joint>
     <joint name="link_3_wrist_joint" type="revolute">
@@ -177,8 +177,8 @@
         <axis xyz="1 0 0.0" />
         <limit lower="-3.14" upper="3.14" effort="100.0" velocity="10.0" />
-        <!-- <dynamics damping="10" friction="10" /> -->
+        <dynamics damping="10" friction="10" />
     </joint>
     <xacro:gripper parent_link="link_3_wrist">
-        <origin xyz="0 0 0.082" rpy="1.5707963 0 0" />
+        <origin xyz="0 -0.085 0" rpy="3.14 0 0" />
     </xacro:gripper>
     <xacro:include filename="visiona_gazebo.xacro" />

File: src/visiona_bridge/urdf/visiona_gazebo.xacro (robot description, xacro)
@@ -23,13 +23,17 @@
     <gazebo reference="gripper_base">
         <material>Gazebo/Green</material>
-        <self_collide>false</self_collide>
+        <self_collide>true</self_collide>
     </gazebo>
     <gazebo reference="left_finger_link">
         <material>Gazebo/Green</material>
-        <self_collide>false</self_collide>
+        <self_collide>true</self_collide>
+        <mu1>1000.0</mu1>
+        <mu2>1000.0</mu2>
     </gazebo>
     <gazebo reference="right_finger_link">
         <material>Gazebo/Green</material>
-        <self_collide>false</self_collide>
+        <self_collide>true</self_collide>
+        <mu1>1000.0</mu1>
+        <mu2>1000.0</mu2>
     </gazebo>
     <xacro:if value="$(arg use_sim)">
