Commit message: merged gazebo with rviz

File: install/visiona_bridge/share/visiona_bridge/urdf/gripper.xacro (robot description, xacro)
@@ -9,10 +9,6 @@
                         scale="0.001 0.001 0.001" />
                 </geometry>
-                <!-- <material name="PLA">
-                    <color rgba="0.0 1.0 0.0 0.5" />
-                    <texture filename="" />
-                </material> -->
             </visual>
-            <collision>
+            <!-- <collision>
                 <origin xyz="0 0 0" rpy="0 0 0" />
                 <geometry>
@@ -20,8 +16,8 @@
                         scale="0.001 0.001 0.001" />
                 </geometry>
-            </collision>
+            </collision> -->
             <inertial>
-                <mass value="0.01" />
-                <inertia ixx="0.001" ixy="0" ixz="0" iyy="0.001" iyz="0" izz="0.001" />
+                <mass value="0.1" />
+                <inertia ixx="0.01" ixy="0" ixz="0" iyy="0.01" iyz="0" izz="0.01" />
             </inertial>
         </link>
@@ -31,9 +27,9 @@
             <xacro:insert_block name="origin_block" />
             <axis xyz="0 1 0.0" />
-            <limit lower="-3.0" upper="3.0" effort="0.0" velocity="0.0" />
+            <limit lower="-3.0" upper="3.0" effort="100.0" velocity="10.0" />
+            <!-- <dynamics damping="10" friction="10" /> -->
         </joint>
         <link name="left_finger_link">
             <visual>
-                <!-- UPDATE THIS: Use the mesh for the left finger/gear -->
                 <origin xyz="0 0 0" rpy="0 0 0" />
                 <geometry>
@@ -41,10 +37,6 @@
                         scale="0.001 0.001 0.001" />
                 </geometry>
-                <!-- <material name="PLA">
-                    <color rgba="0.0 1.0 0.0 0.1" />
-                    <texture filename="" />
-                </material> -->
             </visual>
-            <collision>
+            <!-- <collision>
                 <origin xyz="0 0 0" rpy="0 0 0" />
                 <geometry>
@@ -52,8 +44,8 @@
                         scale="0.001 0.001 0.001" />
                 </geometry>
-            </collision>
+            </collision> -->
             <inertial>
-                <mass value="0.01" />
-                <inertia ixx="0.001" ixy="0" ixz="0" iyy="0.001" iyz="0" izz="0.001" />
+                <mass value="0.1" />
+                <inertia ixx="0.01" ixy="0" ixz="0" iyy="0.01" iyz="0" izz="0.01" />
             </inertial>
         </link>
@@ -65,10 +57,6 @@
                         scale="0.001 0.001 0.001" />
                 </geometry>
-                <!-- <material name="PLA">
-                    <color rgba="0.0 1.0 0.0 0.1" />
-                    <texture filename="" />
-                </material> -->
             </visual>
-            <collision>
+            <!-- <collision>
                 <origin xyz="0 0 0" rpy="0 0 0" />
                 <geometry>
@@ -76,8 +64,8 @@
                         scale="0.001 0.001 0.001" />
                 </geometry>
-            </collision>
+            </collision> -->
             <inertial>
-                <mass value="0.01" />
-                <inertia ixx="0.001" ixy="0" ixz="0" iyy="0.001" iyz="0" izz="0.001" />
+                <mass value="0.1" />
+                <inertia ixx="0.01" ixy="0" ixz="0" iyy="0.01" iyz="0" izz="0.01" />
             </inertial>
         </link>
@@ -85,10 +73,8 @@
             <parent link="gripper_base" />
             <child link="left_finger_link" />
-            <!-- Updated origin from your code -->
             <origin xyz="0.0 0.0 0" rpy="0 0 0" />
-            <!-- Updated axis from your code -->
             <axis xyz="0 0 1" />
-            <!-- Updated limits from your code -->
-            <limit lower="-1.0" upper="1" effort="10" velocity="1.0" />
+            <limit lower="-1.0" upper="1" effort="100.0" velocity="10.0" />
+            <!-- <dynamics damping="10" friction="10" /> -->
         </joint>
         <joint name="right_finger_joint" type="revolute">
@@ -97,6 +83,6 @@
             <origin xyz="0 0 0" rpy="0 0 0" />
             <axis xyz="0 0 1" />
-            <limit lower="-1.0" upper="1" effort="10" velocity="1.0" />
-            <!-- THE MAGIC: This tells this joint to mimic the left one, with a -1 multiplier -->
+            <limit lower="-1.0" upper="1" effort="100.0" velocity="10.0" />
+            <!-- <dynamics damping="10" friction="10" /> -->
             <mimic joint="left_finger_joint" multiplier="-1" offset="0.0" />
         </joint>

File: install/visiona_bridge/share/visiona_bridge/urdf/visiona.urdf.xacro (robot description, xacro)
@@ -1,5 +1,5 @@
 <?xml version="1.0"?>
 <robot xmlns:xacro="http://www.ros.org/wiki/xacro" name="visiona">
-    <!-- Import the gripper macro -->
+    <xacro:arg name="controller_config_path" default="" />
     <xacro:include filename="./gripper.xacro" />
     <link name="world">
@@ -8,6 +8,6 @@
         <inertial>
             <origin xyz="0.0 0.0 0.0" rpy="0.0 0.0 0.0" />
-            <mass value="0.0" />
-            <inertia ixx="0.0" ixy="0.0" ixz="0.0" iyy="0.0" iyz="0.0" izz="0.0" />
+            <mass value="1.0" />
+            <inertia ixx="0.01" ixy="0.0" ixz="0.0" iyy="0.01" iyz="0.0" izz="0.01" />
         </inertial>
         <visual name="base">
@@ -16,13 +16,33 @@
                 <mesh filename="package://visiona_bridge/meshes/base.stl" scale="0.001 0.001 0.001" />
             </geometry>
-            <!-- <material name="PLA">
-                <color rgba="1.0 0.0 0.0 1.0" />
-                <texture filename="" />
-            </material> -->
         </visual>
-        <collision>
-            <origin xyz="0 0 0 " rpy="0 0 0 " />
+        <collision name="base_clyinder">
+            <origin xyz="0 0 0.05 " rpy="0 0 0 " />
             <geometry>
-                <mesh filename="package://visiona_bridge/meshes/base.stl" scale="0.001 0.001 0.001" />
+                <cylinder length="0.1" radius="0.09" />
+            </geometry>
+        </collision>
+        <collision name="logic_box">
+            <origin xyz="0.18 0 0.05 " rpy="0 0 0 " />
+            <geometry>
+                <box size="0.22 0.21 0.1" />
+            </geometry>
+        </collision>
+        <collision name="foot_1">
+            <origin xyz="-0.12 0 0.012 " rpy="0 0 0 " />
+            <geometry>
+                <box size="0.09 0.08 0.026" />
+            </geometry>
+        </collision>
+        <collision name="foot_2">
+            <origin xyz="0 -0.12  0.012 " rpy="0 0 0 " />
+            <geometry>
+                <box size="0.09 0.08 0.026" />
+            </geometry>
+        </collision>
+        <collision name="foot_3">
+            <origin xyz="0 0.12  0.012 " rpy="0 0 0 " />
+            <geometry>
+                <box size="0.09 0.09 0.026" />
             </geometry>
         </collision>
@@ -31,23 +51,18 @@
         <inertial>
             <origin xyz="0.0 0.0 0.0" rpy="0.0 0.0 0.0" />
-            <mass value="0.0" />
-            <inertia ixx="0.0" ixy="0.0" ixz="0.0" iyy="0.0" iyz="0.0" izz="0.0" />
+            <mass value="1.0" />
+            <inertia ixx="0.01" ixy="0.0" ixz="0.0" iyy="0.01" iyz="0.0" izz="0.01" />
         </inertial>
         <visual name="base_link">
-            <origin xyz="0 0 0.067 " rpy="0 0 0 " />
+            <origin xyz="0 0 0.075 " rpy="0 0 0 " />
             <geometry>
                 <mesh filename="package://visiona_bridge/meshes/base_link.stl"
                     scale="0.001 0.001 0.001" />
             </geometry>
-            <!-- <material name="PLA">
-                <color rgba="1.0 0.0 0.0 1.0" />
-                <texture filename="" />
-            </material> -->
         </visual>
         <collision>
-            <origin xyz="0 0 0.067" rpy="0 0 0 " />
+            <origin xyz="-0.005 0 0.14 " rpy="0 0 0 " />
             <geometry>
-                <mesh filename="package://visiona_bridge/meshes/base_link.stl"
-                    scale="0.001 0.001 0.001" />
+                <cylinder length="0.076" radius="0.06" />
             </geometry>
         </collision>
@@ -56,6 +71,6 @@
         <inertial>
             <origin xyz="0 0 0 " rpy="0.0 0.0 0.0" />
-            <mass value="0.0" />
-            <inertia ixx="0.0" ixy="0.0" ixz="0.0" iyy="0.0" iyz="0.0" izz="0.0" />
+            <mass value="1.0" />
+            <inertia ixx="0.01" ixy="0.0" ixz="0.0" iyy="0.01" iyz="0.0" izz="0.01" />
         </inertial>
         <visual name="link_1_shoulder">
@@ -65,14 +80,9 @@
                     scale="0.001 0.001 0.001" />
             </geometry>
-            <!-- <material name="PLA">
-                <color rgba="0.0 1.0 0.0 0.5" />
-                <texture filename="" />
-            </material> -->
         </visual>
         <collision>
-            <origin xyz="0 0 0 " rpy="0 0 0 " />
+            <origin xyz="-0.002 0 0.13" rpy="0 0 0 " />
             <geometry>
-                <mesh filename="package://visiona_bridge/meshes/link_1_shoulder.stl"
-                    scale="0.001 0.001 0.001" />
+                <box size="0.07 0.07 0.165" />
             </geometry>
         </collision>
@@ -81,6 +91,6 @@
         <inertial>
             <origin xyz="0 0 0 " rpy="0.0 0.0 0.0" />
-            <mass value="0.0" />
-            <inertia ixx="0.0" ixy="0.0" ixz="0.0" iyy="0.0" iyz="0.0" izz="0.0" />
+            <mass value="1.0" />
+            <inertia ixx="0.01" ixy="0.0" ixz="0.0" iyy="0.01" iyz="0.0" izz="0.01" />
         </inertial>
         <visual name="link_2_elbow">
@@ -90,14 +100,9 @@
                     scale="0.001 0.001 0.001" />
             </geometry>
-            <!-- <material name="PLA">
-                <color rgba="0.0 1.0 0.0 0.5" />
-                <texture filename="" />
-            </material> -->
         </visual>
         <collision>
-            <origin xyz="0 0 0 " rpy="0 0 0 " />
+            <origin xyz="-0.00 0 0.088" rpy="0 0 0 " />
             <geometry>
-                <mesh filename="package://visiona_bridge/meshes/link_2_elbow.stl"
-                    scale="0.001 0.001 0.001" />
+                <box size="0.027 0.06 0.115" />
             </geometry>
         </collision>
@@ -106,6 +111,6 @@
         <inertial>
             <origin xyz="0 0 0 " rpy="0.0 0.0 0.0" />
-            <mass value="0.0" />
-            <inertia ixx="0.0" ixy="0.0" ixz="0.0" iyy="0.0" iyz="0.0" izz="0.0" />
+            <mass value="1.0" />
+            <inertia ixx="0.01" ixy="0.0" ixz="0.0" iyy="0.01" iyz="0.0" izz="0.01" />
         </inertial>
         <visual name="link_3_wrist">
@@ -115,14 +120,21 @@
                     scale="0.001 0.001 0.001" />
             </geometry>
-            <!-- <material name="PLA">
-                <color rgba="0.0 1.0 0.0 0.5" />
-                <texture filename="" />
-            </material> -->
         </visual>
         <collision>
-            <origin xyz="0 0 0 " rpy="0 0 0 " />
+            <origin xyz="-0.00 0 0.058" rpy="0 0 0 " />
             <geometry>
-                <mesh filename="package://visiona_bridge/meshes/link_3_wrist.stl"
-                    scale="0.001 0.001 0.001" />
+                <box size="0.067 0.06 0.045" />
+            </geometry>
+        </collision>
+        <collision>
+            <origin xyz="-0.027 0 0.003" rpy="0 0 0 " />
+            <geometry>
+                <box size="0.018 0.06 0.06" />
+            </geometry>
+        </collision>
+        <collision>
+            <origin xyz="0.027 0 0.003" rpy="0 0 0 " />
+            <geometry>
+                <box size="0.018 0.06 0.06" />
             </geometry>
         </collision>
@@ -138,13 +150,15 @@
         <parent link="base" />
         <child link="base_link" />
-        <axis xyz="0.0 0.0 1" />
-        <limit lower="-3.14" upper="3.14" effort="0.0" velocity="0.0" />
+        <axis xyz="0.0 0 1" />
+        <limit lower="-3.14" upper="3.14" effort="100.0" velocity="10.0" />
+        <!-- <dynamics damping="10" friction="10" /> -->
     </joint>
     <joint name="link_1_shoulder_joint" type="revolute">
-        <origin xyz="-0.007 0 0.134 " rpy="0.0 0.0 0.0" />
+        <origin xyz="-0.0055 0 0.134 " rpy="0.0 0.0 0.0" />
         <parent link="base_link" />
         <child link="link_1_shoulder" />
         <axis xyz="1 0 0.0" />
-        <limit lower="-1.52" upper="1.52" effort="0.0" velocity="0.0" />
+        <limit lower="-1.52" upper="1.52" effort="100.0" velocity="10.0" />
+        <!-- <dynamics damping="10" friction="10" /> -->
     </joint>
     <joint name="link_2_elbow_joint" type="revolute">
@@ -153,5 +167,6 @@
         <child link="link_2_elbow" />
         <axis xyz="1 0 0.0" />
-        <limit lower="-3.0" upper="3.0" effort="0.0" velocity="0.0" />
+        <limit lower="-3.0" upper="3.0" effort="100.0" velocity="10.0" />
+        <!-- <dynamics damping="10" friction="10" /> -->
     </joint>
     <joint name="link_3_wrist_joint" type="revolute">
@@ -160,40 +175,11 @@
         <child link="link_3_wrist" />
         <axis xyz="1 0 0.0" />
-        <limit lower="-3.0" upper="3.0" effort="0.0" velocity="0.0" />
+        <limit lower="-3.0" upper="3.0" effort="100.0" velocity="10.0" />
+        <!-- <dynamics damping="10" friction="10" /> -->
     </joint>
-    <!-- <joint name="gripper_joint" type="revolute">
-        <origin xyz="0 0 0.082 " rpy="1.5707963 0 0" />
-        <parent link="link_3_wrist" />
-        <child
-            link="gripper_joint" />grip per_joint <axis xyz="0 1 0.0" />
-        <limit lower="-3.0"
-            upper="3.0" effort="0.0" velocity="0.0" />
-    </joint> -->
     <xacro:gripper parent_link="link_3_wrist">
         <origin xyz="0 0 0.082" rpy="1.5707963 0 0" />
     </xacro:gripper>
+    <xacro:include filename="visiona_gazebo.xacro" />
+    <xacro:include filename="visiona.ros2_control.xacro" />
 </robot>
-<!-- <link name="gripper_joint">
-    <inertial>
-        <origin xyz="0 0 0 " rpy="0.0 0.0 0.0" />
-        <mass value="0.0" />
-        <inertia ixx="0.0" ixy="0.0" ixz="0.0" iyy="0.0" iyz="0.0" izz="0.0" />
-    </inertial>
-    <visual name="gripper_joint">
-        <origin xyz="0 0 0 " rpy="0 0 0 " />
-        <geometry>
-            <mesh filename="package://visiona_bridge/meshes/gripper_joint.stl" scale="0.001 0.001 0.001" />
-        </geometry>
-        <material name="PLA">
-                <color rgba="0.0 1.0 0.0 0.5" />
-                <texture filename="" />
-            </material>
-</visual>
-<collision>
-    <origin xyz="0 0 0 " rpy="0 0 0 " />
-    <geometry>
-        <mesh filename="package://visiona_bridge/meshes/gripper_joint.stl" scale="0.001 0.001 0.001" />
-    </geometry>
-</collision>
-</link>
--->

Commit message: feat: Implement Gazebo digital twin synchronization, update URDF mesh paths, and refactor controller configuration.(Sim still needs some Fixing)

File: install/visiona_bridge/share/visiona_bridge/urdf/gripper.xacro (robot description, xacro)
@@ -6,5 +6,5 @@
                 <origin xyz="0 0 0" rpy="0 0 0" />
                 <geometry>
-                    <mesh filename="package://visiona_bridge/meshes/gripper_joint.stl"
+                    <mesh filename="file:///home/farouk/ros2_ws/src/visiona_bridge/meshes/gripper_joint.stl"
                         scale="0.001 0.001 0.001" />
                 </geometry>
@@ -13,5 +13,5 @@
                 <origin xyz="0 0 0" rpy="0 0 0" />
                 <geometry>
-                    <mesh filename="package://visiona_bridge/meshes/gripper_joint.stl"
+                    <mesh filename="file:///home/farouk/ros2_ws/src/visiona_bridge/meshes/gripper_joint.stl"
                         scale="0.001 0.001 0.001" />
                 </geometry>
@@ -34,5 +34,5 @@
                 <origin xyz="0 0 0" rpy="0 0 0" />
                 <geometry>
-                    <mesh filename="package://visiona_bridge/meshes/gripper_left_finger.stl"
+                    <mesh filename="file:///home/farouk/ros2_ws/src/visiona_bridge/meshes/gripper_left_finger.stl"
                         scale="0.001 0.001 0.001" />
                 </geometry>
@@ -41,5 +41,5 @@
                 <origin xyz="0 0 0" rpy="0 0 0" />
                 <geometry>
-                    <mesh filename="package://visiona_bridge/meshes/gripper_left_finger.stl"
+                    <mesh filename="file:///home/farouk/ros2_ws/src/visiona_bridge/meshes/gripper_left_finger.stl"
                         scale="0.001 0.001 0.001" />
                 </geometry>
@@ -54,5 +54,5 @@
                 <origin xyz="0 0 0" rpy="0 0 0" />
                 <geometry>
-                    <mesh filename="package://visiona_bridge/meshes/gripper_right_finger.stl"
+                    <mesh filename="file:///home/farouk/ros2_ws/src/visiona_bridge/meshes/gripper_right_finger.stl"
                         scale="0.001 0.001 0.001" />
                 </geometry>

File: install/visiona_bridge/share/visiona_bridge/urdf/visiona.urdf.xacro (robot description, xacro)
@@ -2,4 +2,5 @@
 <robot xmlns:xacro="http://www.ros.org/wiki/xacro" name="visiona">
     <xacro:arg name="controller_config_path" default="" />
+    <xacro:arg name="use_sim" default="true" />
     <xacro:include filename="./gripper.xacro" />
     <link name="world">
@@ -14,5 +15,5 @@
             <origin xyz="0 0 0 " rpy="0 0 0 " />
             <geometry>
-                <mesh filename="package://visiona_bridge/meshes/base.stl" scale="0.001 0.001 0.001" />
+                <mesh filename="file:///home/farouk/ros2_ws/src/visiona_bridge/meshes/base.stl" scale="0.001 0.001 0.001" />
             </geometry>
         </visual>
@@ -57,5 +58,5 @@
             <origin xyz="0 0 0.075 " rpy="0 0 0 " />
             <geometry>
-                <mesh filename="package://visiona_bridge/meshes/base_link.stl"
+                <mesh filename="file:///home/farouk/ros2_ws/src/visiona_bridge/meshes/base_link.stl"
                     scale="0.001 0.001 0.001" />
             </geometry>
@@ -77,5 +78,5 @@
             <origin xyz="0 0 0 " rpy="0 0 0 " />
             <geometry>
-                <mesh filename="package://visiona_bridge/meshes/link_1_shoulder.stl"
+                <mesh filename="file:///home/farouk/ros2_ws/src/visiona_bridge/meshes/link_1_shoulder.stl"
                     scale="0.001 0.001 0.001" />
             </geometry>
@@ -97,5 +98,5 @@
             <origin xyz="0 0 0 " rpy="0 0 0 " />
             <geometry>
-                <mesh filename="package://visiona_bridge/meshes/link_2_elbow.stl"
+                <mesh filename="file:///home/farouk/ros2_ws/src/visiona_bridge/meshes/link_2_elbow.stl"
                     scale="0.001 0.001 0.001" />
             </geometry>
@@ -117,5 +118,5 @@
             <origin xyz="0 0 0 " rpy="0 0 0 " />
             <geometry>
-                <mesh filename="package://visiona_bridge/meshes/link_3_wrist.stl"
+                <mesh filename="file:///home/farouk/ros2_ws/src/visiona_bridge/meshes/link_3_wrist.stl"
                     scale="0.001 0.001 0.001" />
             </geometry>

File: install/visiona_bridge/share/visiona_bridge/urdf/visiona_gazebo.xacro (robot description, xacro)
@@ -30,16 +30,18 @@
         <self_collide>false</self_collide>
     </gazebo>
-    <gazebo>
-        <plugin name="gazebo_ros_joint_state_publisher"
-            filename="libgazebo_ros_joint_state_publisher.so">
-            <update_rate>20</update_rate>
-            <joint_name>base_link_joint</joint_name>
-            <joint_name>link_1_shoulder_joint</joint_name>
-            <joint_name>link_2_elbow_joint</joint_name>
-            <joint_name>link_3_wrist_joint</joint_name>
-            <joint_name>link_3_wrist_to_gripper_base_joint</joint_name>
-            <joint_name>left_finger_joint</joint_name>
-        </plugin>
-    </gazebo>
+    <xacro:if value="$(arg use_sim)">
+        <gazebo>
+            <plugin name="gazebo_ros_joint_state_publisher"
+                filename="libgazebo_ros_joint_state_publisher.so">
+                <update_rate>20</update_rate>
+                <joint_name>base_link_joint</joint_name>
+                <joint_name>link_1_shoulder_joint</joint_name>
+                <joint_name>link_2_elbow_joint</joint_name>
+                <joint_name>link_3_wrist_joint</joint_name>
+                <joint_name>link_3_wrist_to_gripper_base_joint</joint_name>
+                <joint_name>left_finger_joint</joint_name>
+            </plugin>
+        </gazebo>
+    </xacro:if>
     <gazebo>
         <plugin name="gazebo_ros_joint_pose_trajectory"
@@ -48,9 +50,45 @@
         </plugin>
     </gazebo>
-    <!-- <gazebo>
-        <plugin name="gazebo_ros2_control"
-            filename="libgazebo_ros2_control.so">
-            <parameters>$(arg controller_config_path)</parameters>
-        </plugin>
-    </gazebo> -->
+    <xacro:if value="$(arg use_sim)">
+        <gazebo>
+            <plugin name="gazebo_ros2_control"
+                filename="libgazebo_ros2_control.so">
+                <parameters>$(arg controller_config_path)</parameters>
+            </plugin>
+        </gazebo>
+    </xacro:if>
+    <xacro:unless value="$(arg use_sim)">
+        <gazebo reference="base">
+            <kinematic>true</kinematic>
+            <gravity>false</gravity>
+        </gazebo>
+        <gazebo reference="base_link">
+            <kinematic>true</kinematic>
+            <gravity>false</gravity>
+        </gazebo>
+        <gazebo reference="link_1_shoulder">
+            <kinematic>true</kinematic>
+            <gravity>false</gravity>
+        </gazebo>
+        <gazebo reference="link_2_elbow">
+            <kinematic>true</kinematic>
+            <gravity>false</gravity>
+        </gazebo>
+        <gazebo reference="link_3_wrist">
+            <kinematic>true</kinematic>
+            <gravity>false</gravity>
+        </gazebo>
+        <gazebo reference="gripper_base">
+            <kinematic>true</kinematic>
+            <gravity>false</gravity>
+        </gazebo>
+        <gazebo reference="left_finger_link">
+            <kinematic>true</kinematic>
+            <gravity>false</gravity>
+        </gazebo>
+        <gazebo reference="right_finger_link">
+            <kinematic>true</kinematic>
+            <gravity>false</gravity>
+        </gazebo>
+    </xacro:unless>
 </robot>
