Commit message: test

File: install/visiona_bridge/share/visiona_bridge/urdf/gripper.xacro (robot description, xacro)
@@ -10,5 +10,6 @@
                 </geometry>
             </visual>
-            <!-- <collision>
+            <!-- Collision enabled -->
+            <collision>
                 <origin xyz="0 0 0" rpy="0 0 0" />
                 <geometry>
@@ -16,5 +17,5 @@
                         scale="0.001 0.001 0.001" />
                 </geometry>
-            </collision> -->
+            </collision>
             <inertial>
                 <mass value="0.1" />
@@ -38,5 +39,5 @@
                 </geometry>
             </visual>
-            <!-- <collision>
+            <collision>
                 <origin xyz="0 0 0" rpy="0 0 0" />
                 <geometry>
@@ -44,5 +45,5 @@
                         scale="0.001 0.001 0.001" />
                 </geometry>
-            </collision> -->
+            </collision>
             <inertial>
                 <mass value="0.1" />
@@ -58,11 +59,11 @@
                 </geometry>
             </visual>
-            <!-- <collision>
+            <collision>
                 <origin xyz="0 0 0" rpy="0 0 0" />
                 <geometry>
-                    <mesh filename="package://visiona_bridge/meshes/gripper_right_finger.stl"
+                    <mesh filename="file:///home/farouk/ros2_ws/src/visiona_bridge/meshes/gripper_right_finger.stl"
                         scale="0.001 0.001 0.001" />
                 </geometry>
-            </collision> -->
+            </collision>
             <inertial>
                 <mass value="0.1" />

File: install/visiona_bridge/share/visiona_bridge/urdf/visiona.urdf.xacro (robot description, xacro)
@@ -96,5 +96,5 @@
         </inertial>
         <visual name="link_2_elbow">
-            <origin xyz="0 0 0 " rpy="0 0 0 " />
+            <origin xyz="0 0 0 " rpy="1.57 0 0 " />
             <geometry>
                 <mesh filename="file:///home/farouk/ros2_ws/src/visiona_bridge/meshes/link_2_elbow.stl"
@@ -103,5 +103,5 @@
         </visual>
         <collision>
-            <origin xyz="-0.00 0 0.088" rpy="0 0 0 " />
+            <origin xyz="-0.00 0 0.088" rpy="1.57 0 0 " />
             <geometry>
                 <box size="0.027 0.06 0.115" />
@@ -116,5 +116,5 @@
         </inertial>
         <visual name="link_3_wrist">
-            <origin xyz="0 0 0 " rpy="0 0 0 " />
+            <origin xyz="0 0 0 " rpy="1.57 0 0 " />
             <geometry>
                 <mesh filename="file:///home/farouk/ros2_ws/src/visiona_bridge/meshes/link_3_wrist.stl"
@@ -123,5 +123,5 @@
         </visual>
         <collision>
-            <origin xyz="-0.00 0 0.058" rpy="0 0 0 " />
+            <origin xyz="-0.00 0 0.058" rpy="1.57 0 0 " />
             <geometry>
                 <box size="0.067 0.06 0.045" />
@@ -129,5 +129,5 @@
         </collision>
         <collision>
-            <origin xyz="-0.027 0 0.003" rpy="0 0 0 " />
+            <origin xyz="-0.027 0 0.003" rpy="1.57 0 0 " />
             <geometry>
                 <box size="0.018 0.06 0.06" />
@@ -135,5 +135,5 @@
         </collision>
         <collision>
-            <origin xyz="0.027 0 0.003" rpy="0 0 0 " />
+            <origin xyz="0.027 0 0.003" rpy="1.57 0 0 " />
             <geometry>
                 <box size="0.018 0.06 0.06" />
@@ -160,5 +160,5 @@
         <child link="link_1_shoulder" />
         <axis xyz="1 0 0.0" />
-        <limit lower="-1.52" upper="1.52" effort="100.0" velocity="10.0" />
+        <limit lower="-1.57" upper="1.57" effort="100.0" velocity="10.0" />
         <!-- <dynamics damping="10" friction="10" /> -->
     </joint>
@@ -168,5 +168,5 @@
         <child link="link_2_elbow" />
         <axis xyz="1 0 0.0" />
-        <limit lower="-3.0" upper="3.0" effort="100.0" velocity="10.0" />
+        <limit lower="-3.14" upper="3.14" effort="100.0" velocity="10.0" />
         <!-- <dynamics damping="10" friction="10" /> -->
     </joint>
@@ -176,5 +176,5 @@
         <child link="link_3_wrist" />
         <axis xyz="1 0 0.0" />
-        <limit lower="-3.0" upper="3.0" effort="100.0" velocity="10.0" />
+        <limit lower="-3.14" upper="3.14" effort="100.0" velocity="10.0" />
         <!-- <dynamics damping="10" friction="10" /> -->
     </joint>

File: install/visiona_bridge/share/visiona_bridge/urdf/visiona_gazebo.xacro (robot description, xacro)
@@ -21,10 +21,13 @@
         <self_collide>false</self_collide>
     </gazebo>
-    <gazebo
-        reference="link_3_wrist_to_gripper_base_joint">
+    <gazebo reference="gripper_base">
         <material>Gazebo/Green</material>
         <self_collide>false</self_collide>
     </gazebo>
-    <gazebo reference="left_finger_joint">
+    <gazebo reference="left_finger_link">
+        <material>Gazebo/Green</material>
+        <self_collide>false</self_collide>
+    </gazebo>
+    <gazebo reference="right_finger_link">
         <material>Gazebo/Green</material>
         <self_collide>false</self_collide>
@@ -41,4 +44,15 @@
                 <joint_name>link_3_wrist_to_gripper_base_joint</joint_name>
                 <joint_name>left_finger_joint</joint_name>
+            </plugin>
+        </gazebo>
+        <!-- Mimic Joint Plugin for Right Finger -->
+        <gazebo>
+            <plugin name="mimic_joint_plugin" filename="libgazebo_ros_mimic_joint_plugin.so">
+                <joint>left_finger_joint</joint>
+                <mimicJoint>right_finger_joint</mimicJoint>
+                <multiplier>-1.0</multiplier>
+                <offset>0.0</offset>
+                <sensitiveness>0.0</sensitiveness>
+                <maxEffort>100.0</maxEffort>
             </plugin>
         </gazebo>
