Commit message: feat: Add vision/SLAM packages with LFS for large models

File: install/visiona_bridge/share/visiona_bridge/urdf/gripper.xacro (robot description, xacro)
@@ -1,91 +1 @@
-<?xml version="1.0"?>
-<robot xmlns:xacro="http://www.ros.org/wiki/xacro" name="gripper">
-    <xacro:macro name="gripper" params="parent_link *origin_block">
-        <link name="gripper_base">
-            <visual>
-                <origin xyz="0 0 0" rpy="0 0 0" />
-                <geometry>
-                    <mesh filename="file:///home/farouk/ros2_ws/src/visiona_bridge/meshes/gripper_joint.stl"
-                        scale="0.001 0.001 0.001" />
-                </geometry>
-            </visual>
-            <!-- Collision enabled -->
-            <collision>
-                <origin xyz="0 0 0" rpy="0 0 0" />
-                <geometry>
-                    <mesh filename="file:///home/farouk/ros2_ws/src/visiona_bridge/meshes/gripper_joint.stl"
-                        scale="0.001 0.001 0.001" />
-                </geometry>
-            </collision>
-            <inertial>
-                <mass value="0.1" />
-                <inertia ixx="0.01" ixy="0" ixz="0" iyy="0.01" iyz="0" izz="0.01" />
-            </inertial>
-        </link>
-        <joint name="${parent_link}_to_gripper_base_joint" type="revolute">
-            <parent link="${parent_link}" />
-            <child link="gripper_base" />
-            <xacro:insert_block name="origin_block" />
-            <axis xyz="0 1 0.0" />
-            <limit lower="-3.0" upper="3.0" effort="100.0" velocity="10.0" />
-            <!-- <dynamics damping="10" friction="10" /> -->
-        </joint>
-        <link name="left_finger_link">
-            <visual>
-                <origin xyz="0 0 0" rpy="0 0 0" />
-                <geometry>
-                    <mesh filename="file:///home/farouk/ros2_ws/src/visiona_bridge/meshes/gripper_left_finger.stl"
-                        scale="0.001 0.001 0.001" />
-                </geometry>
-            </visual>
-            <collision>
-                <origin xyz="0 0 0" rpy="0 0 0" />
-                <geometry>
-                    <mesh filename="file:///home/farouk/ros2_ws/src/visiona_bridge/meshes/gripper_left_finger.stl"
-                        scale="0.001 0.001 0.001" />
-                </geometry>
-            </collision>
-            <inertial>
-                <mass value="0.1" />
-                <inertia ixx="0.01" ixy="0" ixz="0" iyy="0.01" iyz="0" izz="0.01" />
-            </inertial>
-        </link>
-        <link name="right_finger_link">
-            <visual>
-                <origin xyz="0 0 0" rpy="0 0 0" />
-                <geometry>
-                    <mesh filename="file:///home/farouk/ros2_ws/src/visiona_bridge/meshes/gripper_right_finger.stl"
-                        scale="0.001 0.001 0.001" />
-                </geometry>
-            </visual>
-            <collision>
-                <origin xyz="0 0 0" rpy="0 0 0" />
-                <geometry>
-                    <mesh filename="file:///home/farouk/ros2_ws/src/visiona_bridge/meshes/gripper_right_finger.stl"
-                        scale="0.001 0.001 0.001" />
-                </geometry>
-            </collision>
-            <inertial>
-                <mass value="0.1" />
-                <inertia ixx="0.01" ixy="0" ixz="0" iyy="0.01" iyz="0" izz="0.01" />
-            </inertial>
-        </link>
-        <joint name="left_finger_joint" type="revolute">
-            <parent link="gripper_base" />
-            <child link="left_finger_link" />
-            <origin xyz="0.0 0.0 0" rpy="0 0 0" />
-            <axis xyz="0 0 1" />
-            <limit lower="-1.0" upper="1" effort="100.0" velocity="10.0" />
-            <!-- <dynamics damping="10" friction="10" /> -->
-        </joint>
-        <joint name="right_finger_joint" type="revolute">
-            <parent link="gripper_base" />
-            <child link="right_finger_link" />
-            <origin xyz="0 0 0" rpy="0 0 0" />
-            <axis xyz="0 0 1" />
-            <limit lower="-1.0" upper="1" effort="100.0" velocity="10.0" />
-            <!-- <dynamics damping="10" friction="10" /> -->
-            <mimic joint="left_finger_joint" multiplier="-1" offset="0.0" />
-        </joint>
-    </xacro:macro>
-</robot>
+/home/farouk/ros2_ws/build/visiona_bridge/urdf/gripper.xacro

File: install/visiona_bridge/share/visiona_bridge/urdf/visiona.ros2_control.xacro (robot description, xacro)
@@ -1,38 +1 @@
-<?xml version="1.0"?>
-<robot xmlns:xacro="http://www.ros.org/wiki/xacro">
-    <ros2_control name="GazeboSystem" type="system">
-        <hardware>
-            <plugin>gazebo_ros2_control/GazeboSystem</plugin>
-        </hardware>
-        <joint name="base_link_joint">
-            <command_interface name="position" />
-            <state_interface name="position" />
-            <state_interface name="velocity" />
-        </joint>
-        <joint name="link_1_shoulder_joint">
-            <command_interface name="position" />
-            <state_interface name="position" />
-            <state_interface name="velocity" />
-        </joint>
-        <joint name="link_2_elbow_joint">
-            <command_interface name="position" />
-            <state_interface name="position" />
-            <state_interface name="velocity" />
-        </joint>
-        <joint name="link_3_wrist_joint">
-            <command_interface name="position" />
-            <state_interface name="position" />
-            <state_interface name="velocity" />
-        </joint>
-        <joint name="link_3_wrist_to_gripper_base_joint">
-            <command_interface name="position" />
-            <state_interface name="position" />
-            <state_interface name="velocity" />
-        </joint>
-        <joint name="left_finger_joint">
-            <command_interface name="position" />
-            <state_interface name="position" />
-            <state_interface name="velocity" />
-        </joint>
-    </ros2_control>
-</robot>
+/home/farouk/ros2_ws/build/visiona_bridge/urdf/visiona.ros2_control.xacro

File: install/visiona_bridge/share/visiona_bridge/urdf/visiona.urdf.xacro (robot description, xacro)
@@ -1,186 +1 @@
-<?xml version="1.0"?>
-<robot xmlns:xacro="http://www.ros.org/wiki/xacro" name="visiona">
-    <xacro:arg name="controller_config_path" default="" />
-    <xacro:arg name="use_sim" default="true" />
-    <xacro:include filename="./gripper.xacro" />
-    <link name="world">
-    </link>
-    <link name="base">
-        <inertial>
-            <origin xyz="0.0 0.0 0.0" rpy="0.0 0.0 0.0" />
-            <mass value="1.0" />
-            <inertia ixx="0.01" ixy="0.0" ixz="0.0" iyy="0.01" iyz="0.0" izz="0.01" />
-        </inertial>
-        <visual name="base">
-            <origin xyz="0 0 0 " rpy="0 0 0 " />
-            <geometry>
-                <mesh filename="file:///home/farouk/ros2_ws/src/visiona_bridge/meshes/base.stl" scale="0.001 0.001 0.001" />
-            </geometry>
-        </visual>
-        <collision name="base_clyinder">
-            <origin xyz="0 0 0.05 " rpy="0 0 0 " />
-            <geometry>
-                <cylinder length="0.1" radius="0.09" />
-            </geometry>
-        </collision>
-        <collision name="logic_box">
-            <origin xyz="0.18 0 0.05 " rpy="0 0 0 " />
-            <geometry>
-                <box size="0.22 0.21 0.1" />
-            </geometry>
-        </collision>
-        <collision name="foot_1">
-            <origin xyz="-0.12 0 0.012 " rpy="0 0 0 " />
-            <geometry>
-                <box size="0.09 0.08 0.026" />
-            </geometry>
-        </collision>
-        <collision name="foot_2">
-            <origin xyz="0 -0.12  0.012 " rpy="0 0 0 " />
-            <geometry>
-                <box size="0.09 0.08 0.026" />
-            </geometry>
-        </collision>
-        <collision name="foot_3">
-            <origin xyz="0 0.12  0.012 " rpy="0 0 0 " />
-            <geometry>
-                <box size="0.09 0.09 0.026" />
-            </geometry>
-        </collision>
-    </link>
-    <link name="base_link">
-        <inertial>
-            <origin xyz="0.0 0.0 0.0" rpy="0.0 0.0 0.0" />
-            <mass value="1.0" />
-            <inertia ixx="0.01" ixy="0.0" ixz="0.0" iyy="0.01" iyz="0.0" izz="0.01" />
-        </inertial>
-        <visual name="base_link">
-            <origin xyz="0 0 0.075 " rpy="0 0 0 " />
-            <geometry>
-                <mesh filename="file:///home/farouk/ros2_ws/src/visiona_bridge/meshes/base_link.stl"
-                    scale="0.001 0.001 0.001" />
-            </geometry>
-        </visual>
-        <collision>
-            <origin xyz="-0.005 0 0.14 " rpy="0 0 0 " />
-            <geometry>
-                <cylinder length="0.076" radius="0.06" />
-            </geometry>
-        </collision>
-    </link>
-    <link name="link_1_shoulder">
-        <inertial>
-            <origin xyz="0 0 0 " rpy="0.0 0.0 0.0" />
-            <mass value="1.0" />
-            <inertia ixx="0.01" ixy="0.0" ixz="0.0" iyy="0.01" iyz="0.0" izz="0.01" />
-        </inertial>
-        <visual name="link_1_shoulder">
-            <origin xyz="0 0 0 " rpy="0 0 0 " />
-            <geometry>
-                <mesh filename="file:///home/farouk/ros2_ws/src/visiona_bridge/meshes/link_1_shoulder.stl"
-                    scale="0.001 0.001 0.001" />
-            </geometry>
-        </visual>
-        <collision>
-            <origin xyz="-0.002 0 0.13" rpy="0 0 0 " />
-            <geometry>
-                <box size="0.07 0.07 0.165" />
-            </geometry>
-        </collision>
-    </link>
-    <link name="link_2_elbow">
-        <inertial>
-            <origin xyz="0 0 0 " rpy="0.0 0.0 0.0" />
-            <mass value="1.0" />
-            <inertia ixx="0.01" ixy="0.0" ixz="0.0" iyy="0.01" iyz="0.0" izz="0.01" />
-        </inertial>
-        <visual name="link_2_elbow">
-            <origin xyz="0 0 0 " rpy="1.57 0 0 " />
-            <geometry>
-                <mesh filename="file:///home/farouk/ros2_ws/src/visiona_bridge/meshes/link_2_elbow.stl"
-                    scale="0.001 0.001 0.001" />
-            </geometry>
-        </visual>
-        <collision>
-            <origin xyz="-0.00 0 0.088" rpy="1.57 0 0 " />
-            <geometry>
-                <box size="0.027 0.06 0.115" />
-            </geometry>
-        </collision>
-    </link>
-    <link name="link_3_wrist">
-        <inertial>
-            <origin xyz="0 0 0 " rpy="0.0 0.0 0.0" />
-            <mass value="1.0" />
-            <inertia ixx="0.01" ixy="0.0" ixz="0.0" iyy="0.01" iyz="0.0" izz="0.01" />
-        </inertial>
-        <visual name="link_3_wrist">
-            <origin xyz="0 0 0 " rpy="1.57 0 0 " />
-            <geometry>
-                <mesh filename="file:///home/farouk/ros2_ws/src/visiona_bridge/meshes/link_3_wrist.stl"
-                    scale="0.001 0.001 0.001" />
-            </geometry>
-        </visual>
-        <collision>
-            <origin xyz="-0.00 0 0.058" rpy="1.57 0 0 " />
-            <geometry>
-                <box size="0.067 0.06 0.045" />
-            </geometry>
-        </collision>
-        <collision>
-            <origin xyz="-0.027 0 0.003" rpy="1.57 0 0 " />
-            <geometry>
-                <box size="0.018 0.06 0.06" />
-            </geometry>
-        </collision>
-        <collision>
-            <origin xyz="0.027 0 0.003" rpy="1.57 0 0 " />
-            <geometry>
-                <box size="0.018 0.06 0.06" />
-            </geometry>
-        </collision>
-    </link>
-    <joint name="base_joint" type="fixed">
-        <origin xyz="0.0 0.0 0.0" rpy="0.0 0.0 0.0" />
-        <parent link="world" />
-        <child link="base" />
-        <axis xyz="0.0 0.0 0.0" />
-    </joint>
-    <joint name="base_link_joint" type="revolute">
-        <origin xyz="0.0 0.0 -0.001" rpy="0.0 0.0 0.0" />
-        <parent link="base" />
-        <child link="base_link" />
-        <axis xyz="0.0 0 1" />
-        <limit lower="-3.14" upper="3.14" effort="100.0" velocity="10.0" />
-        <!-- <dynamics damping="10" friction="10" /> -->
-    </joint>
-    <joint name="link_1_shoulder_joint" type="revolute">
-        <origin xyz="-0.0055 0 0.14 " rpy="0.0 0.0 0.0" />
-        <parent link="base_link" />
-        <child link="link_1_shoulder" />
-        <axis xyz="1 0 0.0" />
-        <limit lower="-1.57" upper="1.57" effort="100.0" velocity="10.0" />
-        <!-- <dynamics damping="10" friction="10" /> -->
-    </joint>
-    <joint name="link_2_elbow_joint" type="revolute">
-        <origin xyz="0 0 0.185 " rpy="0 0 3.14" />
-        <parent link="link_1_shoulder" />
-        <child link="link_2_elbow" />
-        <axis xyz="1 0 0.0" />
-        <limit lower="-3.14" upper="3.14" effort="100.0" velocity="10.0" />
-        <!-- <dynamics damping="10" friction="10" /> -->
-    </joint>
-    <joint name="link_3_wrist_joint" type="revolute">
-        <origin xyz="0 -0.119 0 " rpy="-1.57 0 0" />
-        <parent link="link_2_elbow" />
-        <child link="link_3_wrist" />
-        <axis xyz="1 0 0.0" />
-        <limit lower="-3.14" upper="3.14" effort="100.0" velocity="10.0" />
-        <!-- <dynamics damping="10" friction="10" /> -->
-    </joint>
-    <xacro:gripper parent_link="link_3_wrist">
-        <origin xyz="0 -0.085 0" rpy="3.14 0 0" />
-    </xacro:gripper>
-    <xacro:include filename="visiona_gazebo.xacro" />
-    <xacro:include filename="visiona.ros2_control.xacro" />
-</robot>
+/home/farouk/ros2_ws/build/visiona_bridge/urdf/visiona.urdf.xacro

File: install/visiona_bridge/share/visiona_bridge/urdf/visiona_gazebo.xacro (robot description, xacro)
@@ -1,108 +1 @@
-<?xml version="1.0"?>
-<robot xmlns:xacro="http://www.ros.org/wiki/xacro">
-    <gazebo reference="base">
-        <material>Gazebo/Green</material>
-        <self_collide>false</self_collide>
-    </gazebo>
-    <gazebo reference="base_link">
-        <material>Gazebo/Green</material>
-        <self_collide>false</self_collide>
-    </gazebo>
-    <gazebo reference="link_1_shoulder">
-        <material>Gazebo/Green</material>
-        <self_collide>false</self_collide>
-    </gazebo>
-    <gazebo reference="link_2_elbow">
-        <material>Gazebo/Green</material>
-        <self_collide>false</self_collide>
-    </gazebo>
-    <gazebo reference="link_3_wrist">
-        <material>Gazebo/Green</material>
-        <self_collide>false</self_collide>
-    </gazebo>
-    <gazebo reference="gripper_base">
-        <material>Gazebo/Green</material>
-        <self_collide>false</self_collide>
-    </gazebo>
-    <gazebo reference="left_finger_link">
-        <material>Gazebo/Green</material>
-        <self_collide>false</self_collide>
-    </gazebo>
-    <gazebo reference="right_finger_link">
-        <material>Gazebo/Green</material>
-        <self_collide>false</self_collide>
-    </gazebo>
-    <xacro:if value="$(arg use_sim)">
-        <gazebo>
-            <plugin name="gazebo_ros_joint_state_publisher"
-                filename="libgazebo_ros_joint_state_publisher.so">
-                <update_rate>20</update_rate>
-                <joint_name>base_link_joint</joint_name>
-                <joint_name>link_1_shoulder_joint</joint_name>
-                <joint_name>link_2_elbow_joint</joint_name>
-                <joint_name>link_3_wrist_joint</joint_name>
-                <joint_name>link_3_wrist_to_gripper_base_joint</joint_name>
-                <joint_name>left_finger_joint</joint_name>
-            </plugin>
-        </gazebo>
-        <!-- Mimic Joint Plugin for Right Finger -->
-        <gazebo>
-            <plugin name="mimic_joint_plugin" filename="libgazebo_ros_mimic_joint_plugin.so">
-                <joint>left_finger_joint</joint>
-                <mimicJoint>right_finger_joint</mimicJoint>
-                <multiplier>-1.0</multiplier>
-                <offset>0.0</offset>
-                <sensitiveness>0.0</sensitiveness>
-                <maxEffort>100.0</maxEffort>
-            </plugin>
-        </gazebo>
-    </xacro:if>
-    <gazebo>
-        <plugin name="gazebo_ros_joint_pose_trajectory"
-            filename="libgazebo_ros_joint_pose_trajectory.so">
-            <update_rate>20</update_rate>
-        </plugin>
-    </gazebo>
-    <xacro:if value="$(arg use_sim)">
-        <gazebo>
-            <plugin name="gazebo_ros2_control"
-                filename="libgazebo_ros2_control.so">
-                <parameters>$(arg controller_config_path)</parameters>
-            </plugin>
-        </gazebo>
-    </xacro:if>
-    <xacro:unless value="$(arg use_sim)">
-        <gazebo reference="base">
-            <kinematic>true</kinematic>
-            <gravity>false</gravity>
-        </gazebo>
-        <gazebo reference="base_link">
-            <kinematic>true</kinematic>
-            <gravity>false</gravity>
-        </gazebo>
-        <gazebo reference="link_1_shoulder">
-            <kinematic>true</kinematic>
-            <gravity>false</gravity>
-        </gazebo>
-        <gazebo reference="link_2_elbow">
-            <kinematic>true</kinematic>
-            <gravity>false</gravity>
-        </gazebo>
-        <gazebo reference="link_3_wrist">
-            <kinematic>true</kinematic>
-            <gravity>false</gravity>
-        </gazebo>
-        <gazebo reference="gripper_base">
-            <kinematic>true</kinematic>
-            <gravity>false</gravity>
-        </gazebo>
-        <gazebo reference="left_finger_link">
-            <kinematic>true</kinematic>
-            <gravity>false</gravity>
-        </gazebo>
-        <gazebo reference="right_finger_link">
-            <kinematic>true</kinematic>
-            <gravity>false</gravity>
-        </gazebo>
-    </xacro:unless>
-</robot>
+/home/farouk/ros2_ws/build/visiona_bridge/urdf/visiona_gazebo.xacro

File: src/visiona_bridge/urdf/gripper.xacro (robot description, xacro)
@@ -29,5 +29,5 @@
             <axis xyz="0 1 0.0" />
             <limit lower="-3.0" upper="3.0" effort="100.0" velocity="10.0" />
-            <dynamics damping="10" friction="10" />
+            <dynamics damping="1.0" friction="1.0" />
         </joint>
         <link name="left_finger_link">
@@ -77,5 +77,5 @@
             <axis xyz="0 0 1" />
             <limit lower="-1.0" upper="1" effort="100.0" velocity="10.0" />
-            <dynamics damping="10" friction="10" />
+            <dynamics damping="1.0" friction="1.0" />
         </joint>
         <joint name="right_finger_joint" type="revolute">
@@ -85,5 +85,5 @@
             <axis xyz="0 0 1" />
             <limit lower="-1.0" upper="1" effort="100.0" velocity="10.0" />
-            <dynamics damping="10" friction="10" />
+            <dynamics damping="1.0" friction="1.0" />
             <mimic joint="left_finger_joint" multiplier="-1" offset="0.0" />
         </joint>

File: src/visiona_bridge/urdf/visiona.ros2_control.xacro (robot description, xacro)
@@ -35,4 +35,9 @@
             <state_interface name="velocity" />
         </joint>
+        <joint name="right_finger_joint">
+            <command_interface name="position" />
+            <state_interface name="position" />
+            <state_interface name="velocity" />
+        </joint>
     </ros2_control>
 </robot>

File: src/visiona_bridge/urdf/visiona.urdf.xacro (robot description, xacro)
@@ -152,6 +152,6 @@
         <child link="base_link" />
         <axis xyz="0.0 0 1" />
-        <limit lower="-3.14" upper="3.14" effort="100.0" velocity="10.0" />
-        <dynamics damping="10" friction="10" />
+        <limit lower="0.0" upper="3.14" effort="100.0" velocity="10.0" />
+        <dynamics damping="1.0" friction="1.0" />
     </joint>
     <joint name="link_1_shoulder_joint" type="revolute">
@@ -160,6 +160,6 @@
         <child link="link_1_shoulder" />
         <axis xyz="1 0 0.0" />
-        <limit lower="-1.57" upper="1.57" effort="100.0" velocity="10.0" />
-        <dynamics damping="10" friction="10" />
+        <limit lower="0.0" upper="3.14" effort="100.0" velocity="10.0" />
+        <dynamics damping="1.0" friction="1.0" />
     </joint>
     <joint name="link_2_elbow_joint" type="revolute">
@@ -168,6 +168,6 @@
         <child link="link_2_elbow" />
         <axis xyz="1 0 0.0" />
-        <limit lower="-3.14" upper="3.14" effort="100.0" velocity="10.0" />
-        <dynamics damping="10" friction="10" />
+        <limit lower="0.0" upper="3.14" effort="100.0" velocity="10.0" />
+        <dynamics damping="1.0" friction="1.0" />
     </joint>
     <joint name="link_3_wrist_joint" type="revolute">
@@ -176,6 +176,6 @@
         <child link="link_3_wrist" />
         <axis xyz="1 0 0.0" />
-        <limit lower="-3.14" upper="3.14" effort="100.0" velocity="10.0" />
-        <dynamics damping="10" friction="10" />
+        <limit lower="0.0" upper="3.14" effort="100.0" velocity="10.0" />
+        <dynamics damping="1.0" friction="1.0" />
     </joint>
     <xacro:gripper parent_link="link_3_wrist">

File: src/visiona_bridge/urdf/visiona_gazebo.xacro (robot description, xacro)
@@ -48,15 +48,4 @@
                 <joint_name>link_3_wrist_to_gripper_base_joint</joint_name>
                 <joint_name>left_finger_joint</joint_name>
-            </plugin>
-        </gazebo>
-        <!-- Mimic Joint Plugin for Right Finger -->
-        <gazebo>
-            <plugin name="mimic_joint_plugin" filename="libgazebo_ros_mimic_joint_plugin.so">
-                <joint>left_finger_joint</joint>
-                <mimicJoint>right_finger_joint</mimicJoint>
-                <multiplier>-1.0</multiplier>
-                <offset>0.0</offset>
-                <sensitiveness>0.0</sensitiveness>
-                <maxEffort>100.0</maxEffort>
             </plugin>
         </gazebo>
