Commit message: feat: Add Cartesian controller and command forwarder, update URDF/SRDF joint limits and collision rules, and refine launch configurations for simulation and hardware modes.

File: src/visiona_bridge/urdf/visiona.ros2_control.xacro (robot description, xacro)
@@ -1,7 +1,14 @@
 <?xml version="1.0"?>
 <robot xmlns:xacro="http://www.ros.org/wiki/xacro">
-    <ros2_control name="GazeboSystem" type="system">
+    <xacro:arg name="use_mock_hardware" default="false" />
+    <ros2_control name="VisionaSystem" type="system">
         <hardware>
-            <plugin>gazebo_ros2_control/GazeboSystem</plugin>
+            <xacro:if value="$(arg use_mock_hardware)">
+                <plugin>mock_components/GenericSystem</plugin>
+                <!-- Mock supports position interfacing natively -->
+            </xacro:if>
+            <xacro:unless value="$(arg use_mock_hardware)">
+                <plugin>gazebo_ros2_control/GazeboSystem</plugin>
+            </xacro:unless>
         </hardware>
         <joint name="base_link_joint">

File: src/visiona_bridge/urdf/visiona.urdf.xacro (robot description, xacro)
@@ -2,5 +2,7 @@
 <robot xmlns:xacro="http://www.ros.org/wiki/xacro" name="visiona">
     <xacro:arg name="controller_config_path" default="" />
+    <xacro:arg name="controller_config_path" default="" />
     <xacro:arg name="use_sim" default="true" />
+    <xacro:arg name="use_mock_hardware" default="false" />
     <xacro:include filename="./gripper.xacro" />
     <link name="world">
@@ -156,5 +158,5 @@
         <child link="base_link" />
         <axis xyz="0.0 0 1" />
-        <limit lower="0.0" upper="3.14" effort="100.0" velocity="10.0" />
+        <limit lower="-3.14" upper="3.14" effort="100.0" velocity="10.0" />
         <dynamics damping="1.0" friction="1.0" />
     </joint>
@@ -164,5 +166,5 @@
         <child link="link_1_shoulder" />
         <axis xyz="1 0 0.0" />
-        <limit lower="0.0" upper="3.14" effort="100.0" velocity="10.0" />
+        <limit lower="-3.14" upper="3.14" effort="100.0" velocity="10.0" />
         <dynamics damping="1.0" friction="1.0" />
     </joint>
