Commit message: feat: Update Gazebo plugins, refine Visiona robot URDF joint orientations (griper finger in gazebo not working), relax OpenCV dependency, and add a build script.

File: src/visiona_bridge/urdf/gripper.xacro (robot description, xacro)
@@ -10,5 +10,4 @@
                 </geometry>
             </visual>
-            <!-- Collision enabled -->
             <collision>
                 <origin xyz="0 0 0" rpy="0 0 0" />
@@ -23,4 +22,14 @@
             </inertial>
         </link>
+        <gazebo>
+            <plugin name="mimic_joint_plugin" filename="libgazebo_ros_mimic_joint_plugin.so">
+                <joint>gripper</joint>
+                <mimicJoint>right_finger_joint</mimicJoint>
+                <multiplier>-1.0</multiplier>
+                <offset>0.0</offset>
+                <maxEffort>100.0</maxEffort>
+                <hasPID>false</hasPID>
+            </plugin>
+        </gazebo>
         <joint name="${parent_link}_to_gripper_base_joint" type="revolute">
             <parent link="${parent_link}" />
@@ -71,5 +80,5 @@
             </inertial>
         </link>
-        <joint name="left_finger_joint" type="revolute">
+        <joint name="gripper" type="revolute">
             <parent link="gripper_base" />
             <child link="left_finger_link" />
@@ -77,5 +86,5 @@
             <axis xyz="0 0 1" />
             <limit lower="-1.0" upper="1" effort="100.0" velocity="10.0" />
-            <dynamics damping="1.0" friction="1.0" />
+            <dynamics damping="0.1" friction="0.1" />
         </joint>
         <joint name="right_finger_joint" type="revolute">
@@ -85,6 +94,6 @@
             <axis xyz="0 0 1" />
             <limit lower="-1.0" upper="1" effort="100.0" velocity="10.0" />
-            <dynamics damping="1.0" friction="1.0" />
-            <mimic joint="left_finger_joint" multiplier="-1" offset="0.0" />
+            <dynamics damping="0.1" friction="0.1" />
+            <mimic joint="gripper" multiplier="-1" offset="0.0" />
         </joint>
     </xacro:macro>

File: src/visiona_bridge/urdf/visiona.ros2_control.xacro (robot description, xacro)
@@ -14,4 +14,5 @@
             <state_interface name="position" />
             <state_interface name="velocity" />
+            <param name="initial_position">1.57</param>
         </joint>
         <joint name="link_2_elbow_joint">
@@ -19,4 +20,5 @@
             <state_interface name="position" />
             <state_interface name="velocity" />
+            <param name="initial_position">1.57</param>
         </joint>
         <joint name="link_3_wrist_joint">
@@ -24,4 +26,5 @@
             <state_interface name="position" />
             <state_interface name="velocity" />
+            <param name="initial_position">1.57</param>
         </joint>
         <joint name="link_3_wrist_to_gripper_base_joint">
@@ -29,11 +32,7 @@
             <state_interface name="position" />
             <state_interface name="velocity" />
+            <param name="initial_position">1.57</param>
         </joint>
-        <joint name="left_finger_joint">
-            <command_interface name="position" />
-            <state_interface name="position" />
-            <state_interface name="velocity" />
-        </joint>
-        <joint name="right_finger_joint">
+        <joint name="gripper">
             <command_interface name="position" />
             <state_interface name="position" />

File: src/visiona_bridge/urdf/visiona.urdf.xacro (robot description, xacro)
@@ -148,5 +148,5 @@
     </joint>
     <joint name="base_link_joint" type="revolute">
-        <origin xyz="0.0 0.0 -0.001" rpy="0.0 0.0 0.0" />
+        <origin xyz="0.0 0.0 -0.001" rpy="0.0 0.0 -1.57" />
         <parent link="base" />
         <child link="base_link" />
@@ -156,5 +156,5 @@
     </joint>
     <joint name="link_1_shoulder_joint" type="revolute">
-        <origin xyz="-0.0055 0 0.14 " rpy="0.0 0.0 0.0" />
+        <origin xyz="-0.0055 0 0.14 " rpy="-1.57 0.0 0.0" />
         <parent link="base_link" />
         <child link="link_1_shoulder" />
@@ -164,5 +164,5 @@
     </joint>
     <joint name="link_2_elbow_joint" type="revolute">
-        <origin xyz="0 0 0.185 " rpy="0 0 3.14" />
+        <origin xyz="0 0 0.185 " rpy="-1.57 0 3.14" />
         <parent link="link_1_shoulder" />
         <child link="link_2_elbow" />
@@ -172,5 +172,5 @@
     </joint>
     <joint name="link_3_wrist_joint" type="revolute">
-        <origin xyz="0 -0.119 0 " rpy="-1.57 0 0" />
+        <origin xyz="0 -0.119 0 " rpy="-3.14 0 0" />
         <parent link="link_2_elbow" />
         <child link="link_3_wrist" />
@@ -180,5 +180,5 @@
     </joint>
     <xacro:gripper parent_link="link_3_wrist">
-        <origin xyz="0 -0.085 0" rpy="3.14 0 0" />
+        <origin xyz="0 -0.085 0" rpy="3.14 -1.57 0" />
     </xacro:gripper>
     <xacro:include filename="visiona_gazebo.xacro" />

File: src/visiona_bridge/urdf/visiona_gazebo.xacro (robot description, xacro)
@@ -47,5 +47,5 @@
                 <joint_name>link_3_wrist_joint</joint_name>
                 <joint_name>link_3_wrist_to_gripper_base_joint</joint_name>
-                <joint_name>left_finger_joint</joint_name>
+                <joint_name>gripper</joint_name>
             </plugin>
         </gazebo>

Commit message: feat: Update MoveIt configuration, robot URDF, and RVIZ displays, add camera RVIZ view, and remove test script.

File: src/visiona_bridge/urdf/gripper.xacro (robot description, xacro)
@@ -83,7 +83,7 @@
             <parent link="gripper_base" />
             <child link="left_finger_link" />
-            <origin xyz="0.0 0.0 0" rpy="0 0 0" />
+            <origin xyz="0.0 0.0 0" rpy="0 0 -0.2" />
             <axis xyz="0 0 1" />
-            <limit lower="-1.0" upper="1" effort="100.0" velocity="10.0" />
+            <limit lower="-0.1" upper="0.2" effort="100.0" velocity="10.0" />
             <dynamics damping="0.1" friction="0.1" />
         </joint>
@@ -91,7 +91,7 @@
             <parent link="gripper_base" />
             <child link="right_finger_link" />
-            <origin xyz="0 0 0" rpy="0 0 0" />
+            <origin xyz="0 0 0" rpy="0 0 0.2" />
             <axis xyz="0 0 1" />
-            <limit lower="-1.0" upper="1" effort="100.0" velocity="10.0" />
+            <limit lower="-0.1" upper="0.2" effort="100.0" velocity="10.0" />
             <dynamics damping="0.1" friction="0.1" />
             <mimic joint="gripper" multiplier="-1" offset="0.0" />

File: src/visiona_bridge/urdf/visiona.urdf.xacro (robot description, xacro)
@@ -138,5 +138,5 @@
         <child link="link_1_shoulder" />
         <axis xyz="1 0 0.0" />
-        <limit lower="-3.14" upper="3.14" effort="100.0" velocity="10.0" />
+        <limit lower="0" upper="3.14" effort="100.0" velocity="10.0" />
         <dynamics damping="1.0" friction="1.0" />
     </joint>
@@ -146,5 +146,5 @@
         <child link="link_2_elbow" />
         <axis xyz="1 0 0.0" />
-        <limit lower="-3.14" upper="3.14" effort="100.0" velocity="10.0" />
+        <limit lower="0" upper="3.14" effort="100.0" velocity="10.0" />
         <dynamics damping="1.0" friction="1.0" />
     </joint>
@@ -154,5 +154,5 @@
         <child link="link_3_wrist" />
         <axis xyz="1 0 0.0" />
-        <limit lower="-3.14" upper="3.14" effort="100.0" velocity="10.0" />
+        <limit lower="0" upper="3.14" effort="100.0" velocity="10.0" />
         <dynamics damping="1.0" friction="1.0" />
     </joint>
