Commit message: feat: Add roboticsgroup_upatras_gazebo_plugins package, update Visiona URDF for collision and joint origins, and modify related simulation, bridge, and saved robot positions.

File: src/visiona_bridge/urdf/visiona.urdf.xacro (robot description, xacro)
@@ -102,10 +102,10 @@
             </geometry>
         </visual>
-        <collision>
-            <origin xyz="-0.00 0 0.088" rpy="1.57 0 0 " />
+        <!-- <collision>
+            <origin xyz="0.0 0.0 0.0" rpy="1.57 0 0 " />
             <geometry>
                 <box size="0.027 0.06 0.115" />
             </geometry>
-        </collision>
+        </collision> -->
     </link>
     <link name="link_3_wrist">
@@ -116,5 +116,5 @@
         </inertial>
         <visual name="link_3_wrist">
-            <origin xyz="0 0 0 " rpy="1.57 0 0 " />
+            <origin xyz="0 0.005 0 " rpy="1.57 0 0 " />
             <geometry>
                 <mesh filename="file:///home/farouk/ros2_ws/src/visiona_bridge/meshes/link_3_wrist.stl"
@@ -123,4 +123,10 @@
         </visual>
         <collision>
+            <origin xyz="0.0 -0.03 0.02" rpy="1.57 0 0 " />
+            <geometry>
+                <box size="0.08 0.12 0.12" />
+            </geometry>
+        </collision>
+        <!-- <collision>
             <origin xyz="-0.00 0 0.058" rpy="1.57 0 0 " />
             <geometry>
@@ -139,5 +145,5 @@
                 <box size="0.018 0.06 0.06" />
             </geometry>
-        </collision>
+        </collision> -->
     </link>
     <joint name="base_joint" type="fixed">
@@ -164,5 +170,5 @@
     </joint>
     <joint name="link_2_elbow_joint" type="revolute">
-        <origin xyz="0 0 0.185 " rpy="-1.57 0 3.14" />
+        <origin xyz="0 0 0.185 " rpy="-1.57 0 0" />
         <parent link="link_1_shoulder" />
         <child link="link_2_elbow" />
@@ -172,5 +178,5 @@
     </joint>
     <joint name="link_3_wrist_joint" type="revolute">
-        <origin xyz="0 -0.119 0 " rpy="-3.14 0 0" />
+        <origin xyz="0 -0.119 0 " rpy="0 0 0" />
         <parent link="link_2_elbow" />
         <child link="link_3_wrist" />

File: src/visiona_bridge/urdf/visiona_gazebo.xacro (robot description, xacro)
@@ -37,5 +37,6 @@
         <mu2>1000.0</mu2>
     </gazebo>
-    <xacro:if value="$(arg use_sim)">
+    <xacro:arg name="use_gazebo_joint_pub" default="true" />
+    <xacro:if value="$(arg use_gazebo_joint_pub)">
         <gazebo>
             <plugin name="gazebo_ros_joint_state_publisher"

Commit message: feat: Implement MoveIt! configuration for the Visiona robot and update Gazebo ROS2 Control.

File: src/visiona_bridge/urdf/visiona.urdf.xacro (robot description, xacro)
@@ -102,10 +102,10 @@
             </geometry>
         </visual>
-        <!-- <collision>
+        <collision>
             <origin xyz="0.0 0.0 0.0" rpy="1.57 0 0 " />
             <geometry>
                 <box size="0.027 0.06 0.115" />
             </geometry>
-        </collision> -->
+        </collision>
     </link>
     <link name="link_3_wrist">
@@ -188,4 +188,33 @@
         <origin xyz="0 -0.085 0" rpy="3.14 -1.57 0" />
     </xacro:gripper>
+    <!-- Camera Link -->
+    <link name="camera_link">
+        <visual>
+            <geometry>
+                <box size="0.05 0.05 0.05"/>
+            </geometry>
+            <material name="black">
+                <color rgba="0 0 0 1"/>
+            </material>
+        </visual>
+        <collision>
+            <geometry>
+                <box size="0.05 0.05 0.05"/>
+            </geometry>
+        </collision>
+    </link>
+    <joint name="camera_joint" type="fixed">
+        <parent link="link_3_wrist"/>
+        <child link="camera_link"/>
+        <!-- Adjust origin to place "on top end in the middle" -->
+        <!-- Based on link_3_wrist dimensions, placing it slightly offset -->
+        <origin xyz="0 -0.05 0.1" rpy="0 0 0"/>
+    </joint>
+    <link name="camera_depth_frame"/>
+    <joint name="camera_depth_joint" type="fixed">
+        <parent link="camera_link"/>
+        <child link="camera_depth_frame"/>
+        <origin xyz="0 0 0" rpy="-1.57 0 -1.57"/>
+    </joint>
     <xacro:include filename="visiona_gazebo.xacro" />
     <xacro:include filename="visiona.ros2_control.xacro" />

Commit message: feat: Update robot URDF collision geometries and joint limits, and revise MoveIt SRDF collision matrix and virtual joint.

File: src/visiona_bridge/urdf/visiona.urdf.xacro (robot description, xacro)
@@ -15,5 +15,6 @@
             <origin xyz="0 0 0 " rpy="0 0 0 " />
             <geometry>
-                <mesh filename="file:///home/farouk/ros2_ws/src/visiona_bridge/meshes/base.stl" scale="0.001 0.001 0.001" />
+                <mesh filename="file:///home/farouk/ros2_ws/src/visiona_bridge/meshes/base.stl"
+                    scale="0.001 0.001 0.001" />
             </geometry>
         </visual>
@@ -65,5 +66,5 @@
             <origin xyz="-0.005 0 0.14 " rpy="0 0 0 " />
             <geometry>
-                <cylinder length="0.076" radius="0.06" />
+                <cylinder length="0.076" radius="0.057" />
             </geometry>
         </collision>
@@ -78,12 +79,13 @@
             <origin xyz="0 0 0 " rpy="0 0 0 " />
             <geometry>
-                <mesh filename="file:///home/farouk/ros2_ws/src/visiona_bridge/meshes/link_1_shoulder.stl"
-                    scale="0.001 0.001 0.001" />
-            </geometry>
-        </visual>
-        <collision>
-            <origin xyz="-0.002 0 0.13" rpy="0 0 0 " />
-            <geometry>
-                <box size="0.07 0.07 0.165" />
+                <mesh
+                    filename="file:///home/farouk/ros2_ws/src/visiona_bridge/meshes/link_1_shoulder.stl"
+                    scale="0.001 0.001 0.001" />
+            </geometry>
+        </visual>
+        <collision>
+            <origin xyz="-0.002 0 0.1" rpy="0 0 0 " />
+            <geometry>
+                <box size="0.07 0.07 0.23" />
             </geometry>
         </collision>
@@ -98,12 +100,13 @@
             <origin xyz="0 0 0 " rpy="1.57 0 0 " />
             <geometry>
-                <mesh filename="file:///home/farouk/ros2_ws/src/visiona_bridge/meshes/link_2_elbow.stl"
-                    scale="0.001 0.001 0.001" />
-            </geometry>
-        </visual>
-        <collision>
-            <origin xyz="0.0 0.0 0.0" rpy="1.57 0 0 " />
-            <geometry>
-                <box size="0.027 0.06 0.115" />
+                <mesh
+                    filename="file:///home/farouk/ros2_ws/src/visiona_bridge/meshes/link_2_elbow.stl"
+                    scale="0.001 0.001 0.001" />
+            </geometry>
+        </visual>
+        <collision>
+            <origin xyz="0.0 -0.085 0.0" rpy="1.57 0 0 " />
+            <geometry>
+                <box size="0.027 0.06 0.12" />
             </geometry>
         </collision>
@@ -118,32 +121,27 @@
             <origin xyz="0 0.005 0 " rpy="1.57 0 0 " />
             <geometry>
-                <mesh filename="file:///home/farouk/ros2_ws/src/visiona_bridge/meshes/link_3_wrist.stl"
-                    scale="0.001 0.001 0.001" />
-            </geometry>
-        </visual>
-        <collision>
-            <origin xyz="0.0 -0.03 0.02" rpy="1.57 0 0 " />
-            <geometry>
-                <box size="0.08 0.12 0.12" />
-            </geometry>
-        </collision>
-        <!-- <collision>
-            <origin xyz="-0.00 0 0.058" rpy="1.57 0 0 " />
-            <geometry>
-                <box size="0.067 0.06 0.045" />
-            </geometry>
-        </collision>
-        <collision>
-            <origin xyz="-0.027 0 0.003" rpy="1.57 0 0 " />
-            <geometry>
-                <box size="0.018 0.06 0.06" />
-            </geometry>
-        </collision>
-        <collision>
-            <origin xyz="0.027 0 0.003" rpy="1.57 0 0 " />
-            <geometry>
-                <box size="0.018 0.06 0.06" />
-            </geometry>
-        </collision> -->
+                <mesh
+                    filename="file:///home/farouk/ros2_ws/src/visiona_bridge/meshes/link_3_wrist.stl"
+                    scale="0.001 0.001 0.001" />
+            </geometry>
+        </visual>
+        <collision>
+            <origin xyz="0 -0.03 0" rpy="0 0 0 " />
+            <geometry>
+                <box size="0.068 0.12 0.06" />
+            </geometry>
+        </collision>
+        <collision>
+            <origin xyz="0 -0.075 -0.04" rpy="0 0 0 " />
+            <geometry>
+                <box size="0.04 0.02 0.03" />
+            </geometry>
+        </collision>
+        <collision>
+            <origin xyz="0 -0.06 0.055" rpy="0 0 0 " />
+            <geometry>
+                <box size="0.08 0.04 0.05" />
+            </geometry>
+        </collision>
     </link>
     <joint name="base_joint" type="fixed">
@@ -174,5 +172,5 @@
         <child link="link_2_elbow" />
         <axis xyz="1 0 0.0" />
-        <limit lower="0.0" upper="3.14" effort="100.0" velocity="10.0" />
+        <limit lower="-3.14" upper="3.14" effort="100.0" velocity="10.0" />
         <dynamics damping="1.0" friction="1.0" />
     </joint>
@@ -182,5 +180,5 @@
         <child link="link_3_wrist" />
         <axis xyz="1 0 0.0" />
-        <limit lower="0.0" upper="3.14" effort="100.0" velocity="10.0" />
+        <limit lower="-3.14" upper="3.14" effort="100.0" velocity="10.0" />
         <dynamics damping="1.0" friction="1.0" />
     </joint>
@@ -188,32 +186,30 @@
         <origin xyz="0 -0.085 0" rpy="3.14 -1.57 0" />
     </xacro:gripper>
-    <!-- Camera Link -->
     <link name="camera_link">
         <visual>
             <geometry>
-                <box size="0.05 0.05 0.05"/>
+                <box size="0.09 0.01 0.02" />
             </geometry>
             <material name="black">
-                <color rgba="0 0 0 1"/>
+                <color rgba="0 0 0 1" />
             </material>
         </visual>
         <collision>
             <geometry>
-                <box size="0.05 0.05 0.05"/>
+                <!-- <origin xyz="0 0 0.5" rpy="0 0 0 " /> -->
+                <box size="0.09 0.01 0.02" />
             </geometry>
         </collision>
     </link>
     <joint name="camera_joint" type="fixed">
-        <parent link="link_3_wrist"/>
-        <child link="camera_link"/>
-        <!-- Adjust origin to place "on top end in the middle" -->
-        <!-- Based on link_3_wrist dimensions, placing it slightly offset -->
-        <origin xyz="0 -0.05 0.1" rpy="0 0 0"/>
-    </joint>
-    <link name="camera_depth_frame"/>
+        <parent link="link_3_wrist" />
+        <child link="camera_link" />
+        <origin xyz="0 -0.07 0.069" rpy="0 0 0" />
+    </joint>
+    <link name="camera_depth_frame" />
     <joint name="camera_depth_joint" type="fixed">
-        <parent link="camera_link"/>
-        <child link="camera_depth_frame"/>
-        <origin xyz="0 0 0" rpy="-1.57 0 -1.57"/>
+        <parent link="camera_link" />
+        <child link="camera_depth_frame" />
+        <origin xyz="0 0 0" rpy="0 0 0" />
     </joint>
     <xacro:include filename="visiona_gazebo.xacro" />

Commit message: feat: Implement new firmware, bridge architecture, and GUI with updated MoveIt configurations and launch files.

File: src/visiona_bridge/urdf/visiona.urdf.xacro (robot description, xacro)
@@ -22,31 +22,8 @@
         </visual>
         <collision name="base_clyinder">
-            <origin xyz="0 0 0.05 " rpy="0 0 0 " />
+          <origin xyz="0 0 0 " rpy="0 0 0 " />
             <geometry>
-                <cylinder length="0.1" radius="0.09" />
-            </geometry>
-        </collision>
-        <collision name="logic_box">
-            <origin xyz="0.18 0 0.05 " rpy="0 0 0 " />
-            <geometry>
-                <box size="0.22 0.21 0.1" />
-            </geometry>
-        </collision>
-        <collision name="foot_1">
-            <origin xyz="-0.12 0 0.012 " rpy="0 0 0 " />
-            <geometry>
-                <box size="0.09 0.08 0.026" />
-            </geometry>
-        </collision>
-        <collision name="foot_2">
-            <origin xyz="0 -0.12  0.012 " rpy="0 0 0 " />
-            <geometry>
-                <box size="0.09 0.08 0.026" />
-            </geometry>
-        </collision>
-        <collision name="foot_3">
-            <origin xyz="0 0.12  0.012 " rpy="0 0 0 " />
-            <geometry>
-                <box size="0.09 0.09 0.026" />
+                <mesh filename="file:///home/farouk/ros2_ws/src/visiona_bridge/meshes/base.stl"
+                    scale="0.001 0.001 0.001" />
             </geometry>
         </collision>
@@ -66,7 +43,8 @@
         </visual>
         <collision>
-            <origin xyz="-0.005 0 0.14 " rpy="0 0 0 " />
+            <origin xyz="0 0 0.075 " rpy="0 0 0 " />
             <geometry>
-                <cylinder length="0.076" radius="0.057" />
+                <mesh filename="file:///home/farouk/ros2_ws/src/visiona_bridge/meshes/base_link.stl"
+                    scale="0.001 0.001 0.001" />
             </geometry>
         </collision>
@@ -87,7 +65,9 @@
         </visual>
         <collision>
-            <origin xyz="-0.002 0 0.1" rpy="0 0 0 " />
+            <origin xyz="0 0 0 " rpy="0 0 0 " />
             <geometry>
-                <box size="0.07 0.07 0.23" />
+                <mesh
+                    filename="file:///home/farouk/ros2_ws/src/visiona_bridge/meshes/link_1_shoulder.stl"
+                    scale="0.001 0.001 0.001" />
             </geometry>
         </collision>
@@ -108,7 +88,9 @@
         </visual>
         <collision>
-            <origin xyz="0.0 -0.085 0.0" rpy="1.57 0 0 " />
+            <origin xyz="0 0 0 " rpy="1.57 0 0 " />
             <geometry>
-                <box size="0.027 0.06 0.12" />
+                <mesh
+                    filename="file:///home/farouk/ros2_ws/src/visiona_bridge/meshes/link_2_elbow.stl"
+                    scale="0.001 0.001 0.001" />
             </geometry>
         </collision>
@@ -129,19 +111,9 @@
         </visual>
         <collision>
-            <origin xyz="0 -0.03 0" rpy="0 0 0 " />
+            <origin xyz="0 0.005 0" rpy="1.57 0 0 " />
             <geometry>
-                <box size="0.068 0.12 0.06" />
-            </geometry>
-        </collision>
-        <collision>
-            <origin xyz="0 -0.075 -0.04" rpy="0 0 0 " />
-            <geometry>
-                <box size="0.04 0.02 0.03" />
-            </geometry>
-        </collision>
-        <collision>
-            <origin xyz="0 -0.06 0.055" rpy="0 0 0 " />
-            <geometry>
-                <box size="0.08 0.04 0.05" />
+                <mesh
+                    filename="file:///home/farouk/ros2_ws/src/visiona_bridge/meshes/link_3_wrist.stl"
+                    scale="0.001 0.001 0.001" />
             </geometry>
         </collision>

Commit message: feat: Implement configurable Octomap mapping quality modes, add SLAM setup guide, and update ORB-SLAM integration.

File: src/visiona_bridge/urdf/visiona.urdf.xacro (robot description, xacro)
@@ -179,5 +179,6 @@
         <parent link="link_3_wrist" />
         <child link="camera_link" />
-        <origin xyz="0 -0.07 0.069" rpy="0 0 0" />
+        <!-- Camera pointing DOWN at ground: -90° pitch (around Y axis) -->
+        <origin xyz="0 -0.07 0.069" rpy="0 -1.57 1.57" />
     </joint>
     <link name="camera_depth_frame" />

Commit message: fixed IK movemnts and collosions

File: src/visiona_bridge/urdf/visiona.urdf.xacro (robot description, xacro)
@@ -179,6 +179,5 @@
         <parent link="link_3_wrist" />
         <child link="camera_link" />
-        <!-- Camera pointing DOWN at ground: -90° pitch (around Y axis) -->
-        <origin xyz="0 -0.07 0.069" rpy="0 -1.57 1.57" />
+        <origin xyz="0 -0.07 0.069" rpy="-1.57 0 3.14  " />
     </joint>
     <link name="camera_depth_frame" />
